File: Hardware/pneumatic Backpack v3.0/ADC_pressure.kicad_sch (KiCad schematic)
At the start: 17 parts, among them U1 ABPDLNN100MG2A3, U10 ABPDLNN100MG2A3, U11 ABPDLNN100MG2A3, U12 ABPDLNN100MG2A3, U2 INA332AIDGKR, U5 ABPDLNN100MG2A3, U6 ABPDLNN100MG2A3, U7 ABPDLNN100MG2A3, U8 ABPDLNN100MG2A3, U9 ABPDLNN100MG2A3

Commit message: updated
Parts:
- R3, R4: value 100 -> 100k
Changed lines of the file:
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@@
 		(fields_autoplaced yes)
 		(property "Reference" "R3"
-			(at 19.05 62.2301 0)
-			(effects
-				(font
-					(size 1.27 1.27)
-				)
-				(justify left)
-			)
-		)
-		(property "Value" "100"
-			(at 19.05 59.6901 0)
-			(effects
-				(font
-					(size 1.27 1.27)
-				)
-				(justify left)
+			(at 24.13 59.6899 0)
+			(effects
+				(font
+					(size 1.27 1.27)
+				)
+				(justify right)
+			)
+		)
+		(property "Value" "100k"
+			(at 24.13 62.2299 0)
+			(effects
+				(font
+					(size 1.27 1.27)
+				)
+				(justify right)
 			)
 		)
@@
 		(fields_autoplaced yes)
 		(property "Reference" "R4"
-			(at 19.05 68.5801 0)
-			(effects
-				(font
-					(size 1.27 1.27)
-				)
-				(justify left)
-			)
-		)
-		(property "Value" "100"
-			(at 19.05 66.0401 0)
-			(effects
-				(font
-					(size 1.27 1.27)
-				)
-				(justify left)
-			)
-		)
+			(at 24.13 66.0399 0)
+			(effects
+				(font
+					(size 1.27 1.27)
+				)
+				(justify right)
+			)
+		)
+		(property "Value" "100k"
+			(at 24.13 68.5799 0)
+			(effects
+				(font
+					(size 1.27 1.27)
+				)
+				(justify right)
+			)
+		)
