File: Hardware/pneumatic Backpack v3.0/pneumatic Backpack v3.0.kicad_pcb (KiCad board)
At the start: 2 copper layers, 64 x 73 mm, 41 parts, among them J1 Barrel_Jack_MountingPin, J11 Conn_01x02_Pin, J2 Conn_01x02_Pin, J3 Conn_01x03_Pin, J4 Conn_01x03_Pin, J5 Conn_01x01_Pin, J9 Conn_01x02_Pin, Q1 AO3400A, U1 ABPDLNN100MG2A3, U10 ABPDLNN100MG2A3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

Commit message: updated
Parts:
- added D1: LED, LED_SMD:LED_0805_2012Metric_Pad1.15x1.40mm_HandSolder, F.Cu at (150.1, 76.7)
- added D3: D, Diode_SMD:D_0805_2012Metric_Pad1.15x1.40mm_HandSolder, F.Cu at (150.1, 80.9)
- C1: value 20pf -> 5pf
Routing:
- net Net-(D3-K): track 16.8 -> 26.0 mm
- net Net-(D1-K): track 0.00 -> 2.15 mm
