File: Hardware/pneumatic Backpack v3.0/pneumatic Backpack v3.0.kicad_sch (KiCad schematic)
At the start: 24 parts, among them J1 Barrel_Jack_MountingPin, J11 Conn_01x02_Pin, J2 Conn_01x02_Pin, J3 Conn_01x03_Pin, J4 Conn_01x03_Pin, J5 Conn_01x01_Pin, J9 Conn_01x02_Pin, Q1 AO3400A, U3 R-78C3.3-1.0, U4 R-78C12-1.0

Commit message: updated
Parts:
- added D1: LED, LED_SMD:LED_0805_2012Metric_Pad1.15x1.40mm_HandSolder, symbol Device:LED
- added D3: D, Diode_SMD:D_0805_2012Metric_Pad1.15x1.40mm_HandSolder, symbol Device:D
Connections:
- net +3.3V: now also D1.2 (A)
- net at J3.3 (Pin_3), Q1.3 (D): now also D3.1 (K)
- new net: D1.1 (K), D3.2 (A)
