File: Hardware/pneumatic Backpack v3.1/ADC_diff.kicad_sch (KiCad schematic)
At the start: 25 parts, among them J3 Conn_02x16_Top_Bottom, U3 INA332AIDGKR

Commit message: updated
Parts:
- R21, R22, R23, R24, R25, R26, R27, R28, R29, R30, R31, R32, R33, R34, R35, R36, R37, R38: value 100 -> 100k
Changed lines of the file:
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@@
 			)
 		)
-		(property "Value" "100"
+		(property "Value" "100k"
 			(at 84.328 170.434 0)
 			(effects
@@
 		(fields_autoplaced yes)
 		(property "Reference" "R22"
-			(at 19.05 68.5801 0)
-			(effects
-				(font
-					(size 1.27 1.27)
-				)
-				(justify left)
-			)
-		)
-		(property "Value" "100"
-			(at 19.05 66.0401 0)
-			(effects
-				(font
-					(size 1.27 1.27)
-				)
-				(justify left)
+			(at 24.13 66.0399 0)
+			(effects
+				(font
+					(size 1.27 1.27)
+				)
+				(justify right)
+			)
+		)
+		(property "Value" "100k"
+			(at 24.13 68.5799 0)
+			(effects
+				(font
+					(size 1.27 1.27)
+				)
+				(justify right)
 			)
 		)
@@
 		(fields_autoplaced yes)
 		(property "Reference" "R21"
-			(at 19.05 62.2301 0)
-			(effects
-				(font
-					(size 1.27 1.27)
-				)
-				(justify left)
-			)
-		)
-		(property "Value" "100"
-			(at 19.05 59.6901 0)
-			(effects
-				(font
-					(size 1.27 1.27)
-				)
-				(justify left)
+			(at 24.13 59.6899 0)
+			(effects
+				(font
+					(size 1.27 1.27)
+				)
+				(justify right)
+			)
+		)
+		(property "Value" "100k"
+			(at 24.13 62.2299 0)
+			(effects
+				(font
+					(size 1.27 1.27)
+				)
+				(justify right)
 			)
 		)
@@
 			)
 		)
-		(property "Value" "100"
+		(property "Value" "100k"
 			(at 104.14 170.18 0)
 			(effects
@@
 			)
 		)
-		(property "Value" "100"
+		(property "Value" "100k"
 			(at 97.028 165.862 0)
 			(effects
@@
 			)
 		)
-		(property "Value" "100"
+		(property "Value" "100k"
 			(at 86.614 165.862 0)
 			(effects
@@
 			)
 		)
-		(property "Value" "100"
+		(property "Value" "100k"
 			(at 101.6 165.862 0)
 			(effects
@@
 			)
 		)
-		(property "Value" "100"
+		(property "Value" "100k"
 			(at 78.994 170.434 0)
 			(effects
@@
 			)
 		)
-		(property "Value" "100"
+		(property "Value" "100k"
 			(at 99.06 170.18 0)
 			(effects
@@
 			)
 		)
-		(property "Value" "100"
+		(property "Value" "100k"
 			(at 111.76 165.608 0)
 			(effects
@@
 			)
 		)
-		(property "Value" "100"
+		(property "Value" "100k"
 			(at 76.454 166.116 0)
 			(effects
@@
 			)
 		)
-		(property "Value" "100"
+		(property "Value" "100k"
 			(at 106.68 165.862 0)
 			(effects
@@
 			)
 		)
-		(property "Value" "100"
+		(property "Value" "100k"
 			(at 81.788 166.116 0)
 			(effects
@@
 			)
 		)
-		(property "Value" "100"
+		(property "Value" "100k"
 			(at 109.22 170.18 0)
 			(effects
@@
 			)
 		)
-		(property "Value" "100"
+		(property "Value" "100k"
 			(at 69.85 158.7501 0)
 			(effects
@@
 			)
 		)
-		(property "Value" "100"
+		(property "Value" "100k"
 			(at 94.488 170.18 0)
 			(effects
@@
 			)
 		)
-		(property "Value" "100"
+		(property "Value" "100k"
 			(at 91.948 165.862 0)
 			(effects
@@
 			)
 		)
-		(property "Value" "100"
+		(property "Value" "100k"
 			(at 89.154 170.18 0)
 			(effects
